File: boards/rpi3-isl83488/rpi3-isl83488.kicad_pcb (KiCad board)
At the start: 2 copper layers, 22.9 x 15.2 mm, 10 parts, among them J1 RPi, J2 JST-GH, J3 SERIAL, U1 ISL83488

Commit message: Reduced board width. Reduced size of passives as a result.
Other:
- board text added: "rpi3<>isl83488/90 2020-01 fourside.io"
- board text removed: "rpi3<>isl83488/90 fourside.io"
Changed lines of the file:
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@@
   )
   (setup
-    (last_trace_width 0.3048)
+    (last_trace_width 0.25)
     (user_trace_width 0.1016)
     (user_trace_width 0.1524)
@@
     (pcbplotparams
       (layerselection 0x010fc_ffffffff)
-      (usegerberextensions false)
+      (usegerberextensions true)
       (usegerberattributes false)
-      (usegerberadvancedattributes true)
+      (usegerberadvancedattributes false)
       (creategerberjobfile false)
-      (excludeedgelayer false)
+      (excludeedgelayer true)
       (linewidth 0.150000)
       (plotframeref false)
       (viasonmask false)
       (mode 1)
-      (useauxorigin true)
+      (useauxorigin false)
       (hpglpennumber 1)
       (hpglpenspeed 20)
@@
       (psa4output false)
       (plotreference true)
-      (plotvalue false)
+      (plotvalue true)
       (plotinvisibletext false)
       (padsonsilk false)
@@
   (gr_arc (start 23.368 16.002) (end 23.368 15.24) (angle -90) (layer Edge.Cuts) (width 0.05))
   (gr_arc (start 23.368 29.718) (end 22.606 29.718) (angle -90) (layer Edge.Cuts) (width 0.05))
-  (gr_text "rpi3<>isl83488/90\nfourside.io" (at 44.45 28.194) (layer B.Mask)
+  (gr_text "rpi3<>isl83488/90\n2020-01\nfourside.io" (at 44.45 27.686) (layer B.Mask)
     (effects (font (size 0.9 0.9) (thickness 0.1)) (justify left mirror))
   )
