File: boards/ft2232h-ice40/ft2232h-ice40.kicad_pcb (KiCad board)
At the start: 4 copper layers, 34 x 22.4 mm, 36 parts, among them J1 USB_B_Micro, J2 Conn_01x08, U1 AP7361C_SOT-89-5, U2 FT2232H, X1 ASEM1-12.000MHZ

Commit message: [ft2232h-ice40] Passes DRC.
Other:
- rule trace_min: 0.1524 -> 0.09
- rule via_min_drill: 0.3 -> 0.2
- rule via_min_size: 0.4 -> 0.45
Changed lines of the file:
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@@
     (zone_clearance 0.1524)
     (zone_45_only no)
-    (trace_min 0.1524)
+    (trace_min 0.09)
     (via_size 0.8)
     (via_drill 0.4)
-    (via_min_size 0.4)
-    (via_min_drill 0.3)
+    (via_min_size 0.45)
+    (via_min_drill 0.2)
     (user_via 0.5 0.3)
     (uvia_size 0.3)
@@
     (pad_to_mask_clearance 0.051)
     (solder_mask_min_width 0.25)
+    (pad_to_paste_clearance_ratio -0.15)
     (aux_axis_origin 0 0)
     (visible_elements 7FFFFFFF)
@@
     (descr "LQFP, 64 Pin (https://www.analog.com/media/en/technical-documentation/data-sheets/ad7606_7606-6_7606-4.pdf), generated with kicad-footprint-generator ipc_gullwing_generator.py")
     (tags "LQFP QFP")
-    (solder_paste_ratio -0.2)
+    (solder_paste_ratio -0.15)
     (attr smd)
     (fp_text reference U2 (at 0 0 180) (layer F.SilkS) hide
